File: MainBoard/Version1/MainBoard_v1/MainBoard_v1.kicad_pcb (KiCad board)
At the start: 2 copper layers, 122 x 85.6 mm, 173 parts, among them J1 ILG, J10 SH, J11 SH, J12 SH, J13 FFC, J14 SH, J2 SH, J3 SH, J4 PA, J5 Micro_SD_Card_Det_Hirose_DM3AT, J6 SH, J7 ENC, J8 ENC, J9 PA, Q1 AON7400B, Q10 IRLML6344, Q2 AON7400B, Q3 AON7400B, Q4 AON7400B, Q5 AON7400B, Q6 AON7400B, Q7 2N7002K, Q8 AON7400B, Q9 AON7400B, SW1 SKRPACE010, SW2 SSSS213202, SW3 FR01SC16P-S, SW4 SKRHAAE010, U1 SI7469DP-T1-GE3, U10 DRV8701E, U11 MMC5983MA, U2 LT1963A-TSSOP, U3 TPS62143, U4 ECS-2520S33, U5 INA260, U6 DRV8701E, U7 ICM20648, U8 STM32F469VG, U9 INA260

Commit message: commit
Parts:
- moved D8 116.6 mm to (175.4, 144.4)
- moved D9 114.4 mm to (181.1, 150.9)
- moved R48 114.4 mm to (180.1, 143.2)
- moved R49 114.4 mm to (178.1, 148.2)
- moved R34 78.9 mm to (184.8, 49.4)
- moved R35 78.9 mm to (189.8, 49.2)
- moved R37 78.9 mm to (177.0, 50.0)
- moved R39 78.9 mm to (183.3, 51.5)
- moved R40 78.9 mm to (174.3, 50.5)
- moved R43 78.9 mm to (170.9, 50.8)
- moved R45 78.9 mm to (186.5, 49.1)
- moved R46 78.9 mm to (180.6, 50.0)
- moved R42 78.7 mm to (182.2, 56.1)
- moved R44 75.8 mm to (184.3, 64.0)
- moved R47 75.3 mm to (184.3, 61.4)
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Connections:
- J10 pad 5: (no net) -> Net-(J10-Pad5)
- J13 pad 17: (no net) -> Net-(J13-Pad17)
- J7 pad 1: (no net) -> Net-(J7-Pad1)
- J7 pad 10: (no net) -> Net-(J7-Pad10)
- J7 pad 4: (no net) -> Net-(J7-Pad4)
- J7 pad 5: (no net) -> Net-(J7-Pad5)
- J7 pad 7: (no net) -> Net-(J7-Pad7)
- J7 pad 9: (no net) -> Net-(J7-Pad9)
- J8 pad 1: (no net) -> Net-(J8-Pad1)
- J8 pad 10: (no net) -> Net-(J8-Pad10)
- J8 pad 4: (no net) -> Net-(J8-Pad4)
- J8 pad 5: (no net) -> Net-(J8-Pad5)
- J8 pad 7: (no net) -> Net-(J8-Pad7)
- J8 pad 9: (no net) -> Net-(J8-Pad9)
- SW2 pad 1: (no net) -> Net-(SW2-Pad1)
- U10 pad 11: (no net) -> Net-(U10-Pad11)
- U11 pad 12: (no net) -> Net-(U11-Pad12)
- U11 pad 14: (no net) -> Net-(U11-Pad14)
- U11 pad 15: (no net) -> Net-(U11-Pad15)
- U11 pad 3: (no net) -> Net-(U11-Pad3)
- U11 pad 5: (no net) -> Net-(U11-Pad5)
- U11 pad 6: (no net) -> Net-(U11-Pad6)
- U11 pad 7: (no net) -> Net-(U11-Pad7)
- U11 pad 8: (no net) -> Net-(U11-Pad8)
- U2 pad 11: (no net) -> Net-(U2-Pad11)
- U2 pad 15: (no net) -> Net-(U2-Pad15)
- U2 pad 2: (no net) -> Net-(U2-Pad2)
- U5 pad 13: (no net) -> Net-(U5-Pad13)
- U6 pad 11: (no net) -> Net-(U6-Pad11)
- U7 pad 1: (no net) -> Net-(U7-Pad1)
- U7 pad 11: (no net) -> Net-(U7-Pad11)
- U7 pad 12: (no net) -> Net-(U7-Pad12)
- U7 pad 14: (no net) -> Net-(U7-Pad14)
- U7 pad 15: (no net) -> Net-(U7-Pad15)
- U7 pad 16: (no net) -> Net-(U7-Pad16)
- U7 pad 17: (no net) -> Net-(U7-Pad17)
- U7 pad 19: (no net) -> Net-(U7-Pad19)
- U7 pad 2: (no net) -> Net-(U7-Pad2)
- U7 pad 21: (no net) -> Net-(U7-Pad21)
- U7 pad 3: (no net) -> Net-(U7-Pad3)
- U7 pad 4: (no net) -> Net-(U7-Pad4)
- U7 pad 5: (no net) -> Net-(U7-Pad5)
- U7 pad 6: (no net) -> Net-(U7-Pad6)
- U7 pad 7: (no net) -> Net-(U7-Pad7)
- U8 pad 10: (no net) -> Net-(U8-Pad10)
- U8 pad 34: ENCODER_R_A -> ENCODER_R_B
- U8 pad 36: ENCODER_R_B -> ENCODER_R_A
- U8 pad 4: (no net) -> Net-(U8-Pad4)
- U8 pad 5: (no net) -> Net-(U8-Pad5)
- U8 pad 57: (no net) -> Net-(U8-Pad57)
- U8 pad 58: (no net) -> Net-(U8-Pad58)
- U8 pad 6: (no net) -> Net-(U8-Pad6)
- U8 pad 60: (no net) -> Net-(U8-Pad60)
- U8 pad 61: (no net) -> Net-(U8-Pad61)
- U8 pad 63: (no net) -> Net-(U8-Pad63)
- U8 pad 64: (no net) -> Net-(U8-Pad64)
- U8 pad 93: ESC1_PWM -> ESC2_PWM
- U8 pad 94: ESC2_PWM -> ESC1_PWM
- U9 pad 13: (no net) -> Net-(U9-Pad13)
Routing:
- net GND: track 392.0 -> 481.7 mm, vias 20 -> 22
- net MAKER1: track 0.00 -> 65.2 mm, vias 0 -> 2
- net SW1: track 0.00 -> 62.3 mm, vias 0 -> 1
- net SENSOR_PWM: track 0.00 -> 61.3 mm, vias 0 -> 2
- net SW5: track 0.00 -> 61.3 mm, vias 0 -> 1
- net MAKER2: track 0.00 -> 59.2 mm, vias 0 -> 1
- net SW4: track 0.00 -> 58.9 mm, vias 0 -> 1
- net SW3: track 0.00 -> 58.6 mm, vias 0 -> 1
- net SW2: track 0.00 -> 56.9 mm, vias 0 -> 1
- net AD14: track 0.00 -> 55.6 mm
- net +3V3: track 155.5 -> 210.5 mm
- net AD13: track 0.00 -> 54.0 mm
- net AD12: track 0.00 -> 52.9 mm
- net AD11: track 0.00 -> 51.0 mm
- net R_SW2: track 0.00 -> 49.9 mm
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
Commit message: もう少しで完成
Parts:
- moved C47 76.5 mm to (121.0, 64.5), turned to 180 degrees
- moved C50 74.9 mm to (121.0, 65.9), turned to 180 degrees
- moved C48 74.4 mm to (118.1, 64.5)
- moved C49 72.2 mm to (118.1, 63.1)
- moved C51 70.5 mm to (121.0, 63.1)
- moved SH1 31.7 mm to (153.6, 133.6), turned to 270 degrees
- moved R36 31.0 mm to (167.9, 66.2), turned to 270 degrees
- moved R38 28.9 mm to (164.9, 66.2), turned to 270 degrees
- moved R45 27.0 mm to (163.4, 63.0), turned to 270 degrees
- moved R35 26.6 mm to (169.4, 66.2), turned to 270 degrees
- moved R39 24.7 mm to (163.4, 66.2), turned to 270 degrees
- moved R47 24.0 mm to (160.4, 63.0), turned to 270 degrees
- moved R46 22.8 mm to (161.9, 63.0), turned to 270 degrees
- moved R34 21.8 mm to (170.9, 66.2), turned to 270 degrees
- moved R29 20.4 mm to (159.2, 134.6)
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Connections:
- D8 pad 1: Net-(D8-Pad1) -> GND
- D8 pad 2: LED1 -> Net-(D8-Pad2)
- D9 pad 1: Net-(D9-Pad1) -> GND
- D9 pad 2: LED2 -> Net-(D9-Pad2)
- R48 pad 1: Net-(D8-Pad1) -> LED1
- R48 pad 2: GND -> Net-(D8-Pad2)
- R49 pad 1: Net-(D9-Pad1) -> LED2
- R49 pad 2: GND -> Net-(D9-Pad2)
- RN1 pad 1: SPI_CS -> SPI_MISO
- RN1 pad 2: SPI_SCK -> SPI_MOSI
- RN1 pad 3: SPI_MOSI -> SPI_SCK
- RN1 pad 4: SPI_MISO -> SPI_CS
- SH1 pad 2: EXTRA1 -> EXTRA2
- SH1 pad 3: EXTRA2 -> EXTRA1
- U8 pad 70: LED2 -> LED1
- U8 pad 71: LED1 -> LED2
Routing:
- net +3V3: track 210.5 -> 546.8 mm, vias 7 -> 29
- net GND: track 481.7 -> 758.3 mm, vias 22 -> 43
- net +5V: track 50.6 -> 265.6 mm, vias 2 -> 3
- net SW3: track 58.6 -> 102.9 mm, vias 1 -> 2
- net SW2: track 56.9 -> 99.6 mm, vias 1 -> 2
- net AD10: track 49.2 -> 89.1 mm, vias 0 -> 2
- net AD11: track 51.0 -> 90.7 mm, vias 0 -> 2
- net AD9: track 48.0 -> 87.6 mm, vias 0 -> 2
- net AD8: track 48.4 -> 87.7 mm, vias 0 -> 2
- net AD14: track 55.6 -> 94.6 mm, vias 0 -> 2
- net AD13: track 54.0 -> 92.9 mm, vias 0 -> 2
- net AD12: track 52.9 -> 91.7 mm, vias 0 -> 2
- net AD7: track 48.6 -> 87.3 mm, vias 0 -> 2
- net SW1: track 62.3 -> 94.8 mm, vias 1 -> 2
- net SW4: track 58.9 -> 88.7 mm, vias 1 -> 2
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