File: MainBoard/Version1/MainBoard_v1/MainBoard_v1.sch (KiCad schematic (older format))
At the start: 165 parts, among them J1 ILG, J10 SH, J11 SH, J12 SH, J13 FFC, J14 SH, J2 SH, J3 SH, J4 PA, J5 Micro_SD_Card_Det_Hirose_DM3AT, J6 SH, J7 ENC, J8 ENC, J9 PA, Q1 AON7400B, Q10 IRLML6344, Q2 AON7400B, Q3 AON7400B, Q4 AON7400B, Q5 AON7400B, Q6 AON7400B, Q7 2N7002K, Q8 AON7400B, Q9 AON7400B, SW1 SKRPACE010, SW2 SSSS213202, SW3 FR01SC16P-S, SW4 SKRHAAE010, U1 SI7469DP-T1-GE3, U10 DRV8701E, U11 MMC5983MA, U2 LT1963A-TSSOP, U3 TPS62143, U4 ECS-2520S33, U5 INA260, U6 DRV8701E, U7 ICM20648, U8 STM32F469VG, U9 INA260

Commit message: commit
Connections:
- net ENCODER_R_A: now also U8.36 (PE11); no longer U8.34 (PE9)
- net ENCODER_R_B: now also U8.34 (PE9); no longer U8.36 (PE11)
- net ESC1_PWM: now also U8.94 (PB5); no longer U8.93 (PB4)
- net ESC2_PWM: now also U8.93 (PB4); no longer U8.94 (PB5)
Changed lines of the file:
@@
 Text GLabel 5450 4300 2    50   Input ~ 0
 LED_B
+Text GLabel 3550 6900 3    50   Input ~ 0
+ENCODER_R_A
 Text GLabel 3350 6900 3    50   Input ~ 0
-ENCODER_R_A
-Text GLabel 3550 6900 3    50   Input ~ 0
 ENCODER_R_B
 Text GLabel 4150 6900 3    50   Input ~ 0
@@
 Text GLabel 3450 3500 1    50   Input ~ 0
 SW1
+Text GLabel 3150 3500 1    50   Input ~ 0
+ESC1_PWM
 Text GLabel 3250 3500 1    50   Input ~ 0
-ESC1_PWM
-Text GLabel 3150 3500 1    50   Input ~ 0
 ESC2_PWM
 Text GLabel 3050 3500 1    50   Input ~ 0

Commit message: もう少しで完成
Connections:
- net EXTRA1: now also SH1.3 (Pin_3); no longer SH1.2 (Pin_2)
- net EXTRA2: now also SH1.2 (Pin_2); no longer SH1.3 (Pin_3)
- net GND: now also D8.1 (K), D9.1 (K); no longer R48.2, R49.2
- net LED1: now also R48.1, U8.70 (PA8); no longer D8.2 (A), U8.71 (PA9)
- net LED2: now also R49.1, U8.71 (PA9); no longer D9.2 (A), U8.70 (PA8)
- net SPI_CS: now also RN1.4 (R4.1); no longer RN1.1 (R1.1)
- net SPI_MISO: now also RN1.1 (R1.1); no longer RN1.4 (R4.1)
- net SPI_MOSI: now also RN1.2 (R2.1); no longer RN1.3 (R3.1)
- net SPI_SCK: now also RN1.3 (R3.1); no longer RN1.2 (R2.1)
- new net: D8.2 (A), R48.2
- new net: D9.2 (A), R49.2
Other:
- moved on the sheet: D8, D9, R48, R49
Changed lines of the file:
@@
 Text GLabel 5450 4900 2    50   Input ~ 0
 ENCODER_L_B
-Text GLabel 5450 4400 2    50   Input ~ 0
-LED1
 Text GLabel 5450 4500 2    50   Input ~ 0
+LED1
+Text GLabel 5450 4400 2    50   Input ~ 0
 LED2
 Text GLabel 4550 3500 1    50   Input ~ 0
@@
 NoConn ~ 7350 3700
 $Comp
-L Device:R_Pack04 RN1
-U 1 1 5F39619A
-P 6800 3550
-F 0 "RN1" H 6988 3596 50  0000 L CNN
-F 1 "4.7k" H 6988 3505 50  0000 L CNN
-F 2 "Resistors_SMD:R_Array_Convex_4x1206" V 7075 3550 50  0001 C CNN
-F 3 "~" H 6800 3550 50  0001 C CNN
-	1    6800 3550
-	1    0    0    -1
-$EndComp
-$Comp
 L Device:C_Small C22
 U 1 1 5F3D9C99
@@
 SPI_CS
 Wire Wire Line
-	6550 4000 6600 4000
-Wire Wire Line
-	7350 4100 6700 4100
-Wire Wire Line
-	6550 4200 6800 4200
-Wire Wire Line
-	6550 4300 6900 4300
-Wire Wire Line
 	7500 4300 7500 4800
 Wire Wire Line
@@
 Wire Wire Line
 	8900 4000 8850 4000
-Wire Wire Line
-	6600 3750 6600 4000
-Connection ~ 6600 4000
-Wire Wire Line
-	6600 4000 7350 4000
-Wire Wire Line
-	6700 3750 6700 4100
-Connection ~ 6700 4100
-Wire Wire Line
-	6700 4100 6550 4100
-Wire Wire Line
-	6800 3750 6800 4200
-Connection ~ 6800 4200
-Wire Wire Line
-	6800 4200 7350 4200
-Wire Wire Line
-	6900 3750 6900 4300
-Connection ~ 6900 4300
-Wire Wire Line
-	6900 4300 7500 4300
 $Comp
 L power:+3.3V #PWR021
@@
 Wire Wire Line
 	6300 9200 6300 9250
-Text GLabel 6250 9900 0    50   Input ~ 0
-EXTRA1
 Text GLabel 6250 10000 0    50   Input ~ 0
+EXTRA1
+Text GLabel 6250 9900 0    50   Input ~ 0
 EXTRA2
 $Comp
@@
 L Device:LED_Small_ALT D8
 U 1 1 61039744
-P 1150 10300
+P 1150 10550
 AR Path="/61039744" Ref="D8"  Part="1"
 AR Path="/5F238A80/61039744" Ref="D?"  Part="1"
-F 0 "D8" V 1150 10500 50  0000 R CNN
-F 1 "OSTG1608C1A" V 1650 10500 50  0000 R CNN
-F 2 "LEDs:LED_0603" V 1150 10300 50  0001 C CNN
-F 3 "~" V 1150 10300 50  0001 C CNN
-	1    1150 10300
+F 0 "D8" V 1150 10750 50  0000 R CNN
+F 1 "OSTG1608C1A" V 1650 10750 50  0000 R CNN
+F 2 "LEDs:LED_0603" V 1150 10550 50  0001 C CNN
+F 3 "~" V 1150 10550 50  0001 C CNN
+	1    1150 10550
 	0    -1   -1   0
 $EndComp
@@
 L Device:LED_Small_ALT D9
 U 1 1 6103974A
-P 1450 10300
+P 1450 10550
 AR Path="/6103974A" Ref="D9"  Part="1"
 AR Path="/5F238A80/6103974A" Ref="D?"  Part="1"
-F 0 "D9" V 1450 10250 50  0000 R CNN
-F 1 "OSTG1608C1A" V 1850 10550 50  0000 R CNN
-F 2 "LEDs:LED_0603" V 1450 10300 50  0001 C CNN
-F 3 "~" V 1450 10300 50  0001 C CNN
-	1    1450 10300
+F 0 "D9" V 1450 10500 50  0000 R CNN
+F 1 "OSTG1608C1A" V 1850 10800 50  0000 R CNN
+F 2 "LEDs:LED_0603" V 1450 10550 50  0001 C CNN
+F 3 "~" V 1450 10550 50  0001 C CNN
+	1    1450 10550
 	0    -1   -1   0
 $EndComp
@@
 L Device:R_Small R48
 U 1 1 61039762
-P 1150 10550
+P 1150 10300
 AR Path="/61039762" Ref="R48"  Part="1"
 AR Path="/5F238A80/61039762" Ref="R?"  Part="1"
-F 0 "R48" H 1209 10596 50  0000 L CNN
-F 1 "390" H 1200 10500 50  0000 L CNN
-F 2 "Resistors_SMD:R_0603" H 1150 10550 50  0001 C CNN
-F 3 "~" H 1150 10550 50  0001 C CNN
-	1    1150 10550
+F 0 "R48" H 1209 10346 50  0000 L CNN
+F 1 "390" H 1200 10250 50  0000 L CNN
+F 2 "Resistors_SMD:R_0603" H 1150 10300 50  0001 C CNN
+F 3 "~" H 1150 10300 50  0001 C CNN
+	1    1150 10300
 	-1   0    0    -1
 $EndComp
@@
 L Device:R_Small R49
 U 1 1 61039768
-P 1450 10550
+P 1450 10300
 AR Path="/61039768" Ref="R49"  Part="1"
 AR Path="/5F238A80/61039768" Ref="R?"  Part="1"
-F 0 "R49" H 1509 10596 50  0000 L CNN
-F 1 "390" H 1500 10500 50  0000 L CNN
-F 2 "Resistors_SMD:R_0603" H 1450 10550 50  0001 C CNN
-F 3 "~" H 1450 10550 50  0001 C CNN
-	1    1450 10550
+F 0 "R49" H 1509 10346 50  0000 L CNN
+F 1 "390" H 1500 10250 50  0000 L CNN
+F 2 "Resistors_SMD:R_0603" H 1450 10300 50  0001 C CNN
+F 3 "~" H 1450 10300 50  0001 C CNN
+	1    1450 10300
 	-1   0    0    -1
 $EndComp
@@
 NoConn ~ 2050 4400
 NoConn ~ 2050 4500
+$Comp
+L Device:R_Pack04 RN1
+U 1 1 5F39619A
+P 6800 3550
+F 0 "RN1" H 6988 3596 50  0000 L CNN
+F 1 "4.7k" H 6988 3505 50  0000 L CNN
+F 2 "Resistors_SMD:R_Array_Convex_4x1206" V 7075 3550 50  0001 C CNN
+F 3 "~" H 6800 3550 50  0001 C CNN
+	1    6800 3550
+	1    0    0    -1
+$EndComp
+Wire Wire Line
+	6550 4300 6600 4300
+Wire Wire Line
+	6900 3750 6900 4000
+Connection ~ 6700 4200
+Wire Wire Line
+	6700 4200 7350 4200
+Connection ~ 6800 4100
+Wire Wire Line
+	6800 4100 7350 4100
+Connection ~ 6900 4000
+Wire Wire Line
+	6900 4000 7350 4000
+Wire Wire Line
+	6550 4200 6700 4200
+Wire Wire Line
+	6550 4000 6900 4000
+Wire Wire Line
+	6800 3750 6800 4100
+Wire Wire Line
+	6550 4100 6800 4100
+Wire Wire Line
+	6700 3750 6700 4200
+Wire Wire Line
+	6600 3750 6600 4300
+Connection ~ 6600 4300
+Wire Wire Line
+	6600 4300 7500 4300
 $EndSCHEMATC
