File: FollowingSensor/FollowingSensor1.0/FollowingSensor1.0.kicad_pcb (KiCad board)
At the start: 2 copper layers, 106.9 x 42.1 mm, 33 parts, among them J1 Conn_01x18, Q1 TEMT7100X01, Q10 TEMT7100X01, Q11 TEMT7100X01, Q12 TEMT7100X01, Q13 TEMT7100X01, Q14 TEMT7100X01, Q2 TEMT7100X01, Q3 TEMT7100X01, Q4 TEMT7100X01, Q5 TEMT7100X01, Q6 TEMT7100X01, Q7 TEMT7100X01, Q8 TEMT7100X01, Q9 TEMT7100X01

Commit message: LinesensorUpdate
Parts:
- removed REF** (x2): MountingHole_2.2mm_M2, MountingHole:MountingHole_2.2mm_M2
- moved Q14 31.6 mm to (189.2, 91.5)
- moved Q13 27.8 mm to (183.9, 85.4)
- moved Q9 25.5 mm to (149.2, 72.4)
- moved Q11 24.1 mm to (167.0, 74.1)
- moved Q10 21.1 mm to (157.8, 71.4)
- moved Q12 20.9 mm to (176.1, 79.2)
- moved Q8 19.2 mm to (149.2, 68.5)
Other:
- board size 106.9 x 42.1 mm -> 108.6 x 46.3 mm

Commit message: sensor on the way
Parts:
- moved Q9 51.2 mm to (158.4, 22.0)
- moved Q10 8.61 mm to (149.2, 71.7)
- moved Q11 2.97 mm to (169.5, 75.7), turned to 341 degrees
- moved Q12 1.58 mm to (177.6, 79.7), turned to 331 degrees
- moved Q14 1.34 mm to (190.4, 92.1), turned to 311 degrees
- moved Q13 1.06 mm to (184.6, 86.2), turned to 321 degrees
Other:
- board size 108.6 x 46.3 mm -> 253.6 x 86.9 mm

Commit message: placement phototransister
Parts:
- removed the Q10 at (149.2, 71.7)
- removed the Q9 at (158.4, 22.0)
- added D11: SIR19-21C/TR8, Footprint:SIR19-21C, B.Cu at (208.7, 89.9)
- added D2: SIR19-21C/TR8, Footprint:SIR19-21C, B.Cu at (214.8, 87.5)
- added D4: SIR19-21C/TR8, Footprint:SIR19-21C, B.Cu at (209.3, 95.7)
- added D9: SIR19-21C/TR8, Footprint:SIR19-21C, B.Cu at (214.9, 91.3)
- added Q12: TEMT7100X01, Footprint:TEMT7100X01, B.Cu at (181.5, 82.8)
- added Q13: TEMT7100X01, Footprint:TEMT7100X01, B.Cu at (187.6, 88.7)
- added R10: R, Resistor_SMD:R_0603_1608Metric, F.Cu at (200.9, 77.2)
- added R11: R, Resistor_SMD:R_0603_1608Metric, F.Cu at (204.9, 74.7)
- added R12: R, Resistor_SMD:R_0603_1608Metric, F.Cu at (200.9, 79.7)
- added R9: R, Resistor_SMD:R_0603_1608Metric, F.Cu at (200.9, 74.7)
- D1, D3, Q7, Q8: moved to B.Cu
- D10: renamed from D5; moved to B.Cu
- D12: renamed from D8; moved to B.Cu
- D5: renamed from D2; moved to B.Cu
- D6: renamed from D4; moved to B.Cu
- D7: renamed from D6; moved to B.Cu
- D8: renamed from D7; moved to B.Cu
- Q1: renamed from Q2; moved to B.Cu
- Q10: renamed from Q12; moved to B.Cu
- Q11: renamed from Q14; moved to B.Cu
- Q14: renamed from Q13; moved to B.Cu
- Q2: renamed from Q4; moved to B.Cu
- Q3: renamed from Q6; moved to B.Cu
- Q4: renamed from Q1; moved to B.Cu
- Q5: renamed from Q3; moved to B.Cu
- Q6: renamed from Q5; moved to B.Cu
- Q9: renamed from Q11; moved to B.Cu
- moved Q4 42.6 mm to (125.6, 78.0), turned to 29.3 degrees
- moved Q3 35.1 mm to (118.5, 82.8), turned to 39 degrees
- moved Q5 32.3 mm to (133.3, 74.5), turned to 19.5 degrees
- moved D12 30.8 mm to (194.2, 99.2)
- moved D8 27.0 mm to (188.9, 91.0)
- moved Q6 26.4 mm to (141.5, 72.4), turned to 9.8 degrees
- moved Q2 25.5 mm to (112.4, 88.7), turned to 48.8 degrees
- moved Q7 24.6 mm to (149.2, 69.6)
- moved Q11 21.3 mm to (174.4, 78.0), turned to 330.7 degrees
- moved D7 19.6 mm to (171.2, 72.9)
- moved Q1 18.9 mm to (107.4, 95.5), turned to 58.5 degrees
- moved D10 17.8 mm to (154.9, 69.4)
- moved Q14 12.3 mm to (192.6, 95.5), turned to 301.5 degrees
- moved Q10 12.1 mm to (166.7, 74.5), turned to 340.5 degrees
- moved Q9 11.5 mm to (158.5, 72.4), turned to 350.2 degrees
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- renumbered R3 to R2, R2 to R3, R6 to R5, R7 to R6, R5 to R7

Commit message: following sensor designed
Parts:
- added C1: 1u, Capacitor_SMD:C_0603_1608Metric, B.Cu at (148.4, 82.0)
- R1: moved to B.Cu
- R10: renamed from R7; moved to B.Cu
- R11: renamed from R12; moved to B.Cu
- R12: renamed from R8; moved to B.Cu
- R2: renamed from R9; moved to B.Cu
- R3: renamed from R2; moved to B.Cu
- R4: renamed from R11; moved to B.Cu
- R5: renamed from R3; moved to B.Cu
- R6: renamed from R4; moved to B.Cu
- R7: renamed from R5; moved to B.Cu
- R8: renamed from R6; moved to B.Cu
- R9: renamed from R10; moved to B.Cu
- moved D2 99.5 mm to (115.3, 85.6), turned to 43.9 degrees
- moved R2 84.8 mm to (117.1, 87.4), turned to 43.9 degrees
- moved D4 82.3 mm to (129.4, 76.1), turned to 24.4 degrees
- moved R4 74.6 mm to (130.4, 78.4), turned to 24.4 degrees
- moved D9 46.8 mm to (170.6, 76.1), turned to 335.7 degrees
- moved D5 41.4 mm to (137.4, 73.3), turned to 14.6 degrees
- moved R8 40.5 mm to (162.0, 75.7), turned to 345.4 degrees
- moved R5 39.9 mm to (138.0, 75.7), turned to 14.6 degrees
- moved R10 39.5 mm to (176.6, 82.3), turned to 325.9 degrees
- moved R7 32.4 mm to (154.0, 74.3), turned to 355.1 degrees
- moved R12 31.7 mm to (188.2, 93.5), turned to 306.4 degrees
- moved D8 31.7 mm to (162.6, 73.3), turned to 345.4 degrees
- moved R9 31.3 mm to (169.6, 78.4), turned to 335.7 degrees
- moved R6 28.6 mm to (146.0, 74.3), turned to 4.9 degrees
- moved D10 25.6 mm to (178.1, 80.3), turned to 325.9 degrees
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Connections:
- J1 pad 1: +3V3 -> GND
- J1 pad 10: AD9 -> AD8
- J1 pad 11: AD10 -> AD7
- J1 pad 12: AD11 -> AD6
- J1 pad 13: AD12 -> AD5
- J1 pad 14: AD13 -> AD4
- J1 pad 15: AD14 -> AD3
- J1 pad 16: SENSOR_PULSE -> AD2
- J1 pad 17: Net-(J1-Pad17) -> AD1
- J1 pad 18: GND -> +3V3
- J1 pad 2: AD1 -> Net-(J1-Pad2)
- J1 pad 3: AD2 -> SENSOR_PULSE
- J1 pad 4: AD3 -> AD14
- J1 pad 5: AD4 -> AD13
- J1 pad 6: AD5 -> AD12
- J1 pad 7: AD6 -> AD11
- J1 pad 8: AD7 -> AD10
- J1 pad 9: AD8 -> AD9
Routing:
- net SENSOR_PULSE: track 0.00 -> 159.9 mm, vias 0 -> 3
- net GND: track 0.00 -> 150.2 mm, vias 0 -> 1
- net +3V3: track 0.00 -> 133.4 mm, vias 0 -> 13
- net AD1: track 0.00 -> 48.0 mm, vias 0 -> 1
- net AD14: track 0.00 -> 47.9 mm, vias 0 -> 1
- net AD2: track 0.00 -> 42.6 mm, vias 0 -> 1
- net AD13: track 0.00 -> 41.0 mm, vias 0 -> 1
- net AD3: track 0.00 -> 34.3 mm, vias 0 -> 1
- net AD12: track 0.00 -> 33.7 mm, vias 0 -> 1
- net AD11: track 0.00 -> 26.1 mm, vias 0 -> 1
- net AD4: track 0.00 -> 25.3 mm, vias 0 -> 1
- net AD5: track 0.00 -> 18.8 mm, vias 0 -> 1
- net AD10: track 0.00 -> 18.5 mm, vias 0 -> 1
- net AD6: track 0.00 -> 13.2 mm, vias 0 -> 1
- net AD9: track 0.00 -> 11.9 mm, vias 0 -> 1
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- added copper zone on B.Cu, net GND
- added copper zone on F.Cu, net GND
Other:
- board size 253.6 x 86.9 mm -> 101.6 x 33.9 mm
