File: FollowingSensor/FollowingSensor1.0/FollowingSensor1.0.kicad_pcb (KiCad board)
At the start: 2 copper layers, 101.6 x 33.9 mm, 41 parts, among them J1 Conn_01x18, Q1 TEMT7100X01, Q10 TEMT7100X01, Q11 TEMT7100X01, Q12 TEMT7100X01, Q13 TEMT7100X01, Q14 TEMT7100X01, Q2 TEMT7100X01, Q3 TEMT7100X01, Q4 TEMT7100X01, Q5 TEMT7100X01, Q6 TEMT7100X01, Q7 TEMT7100X01, Q8 TEMT7100X01, Q9 TEMT7100X01

Commit message: fixed
Routing:
- net GND: vias 6 -> 7

Commit message: fixed
Routing:
- net GND: vias 7 -> 16
